Commit message: make signifincantly simpler urdf bounding boxes

File: rerun_arm/robot.urdf (robot description, URDF)
Before this commit: robot henry-robot, 8 links, 7 joints
Links:
- link base: geometry collision box size=0.10 0.10 0.07; visual mesh filename=assets/base.stl
- link distal_arm: geometry collision box size=0.14 0.04 0.04; visual mesh filename=assets/distal_arm.stl
- link jaw: geometry collision box size=0.08 0.015 0.05; visual mesh filename=assets/jaw.stl
- link jaw_base: geometry collision box size=0.05 0.05 0.1; visual mesh filename=assets/jaw_base.stl
- link proximal_arm: geometry collision box size=0.13 0.04 0.04; visual mesh filename=assets/proximal_arm.stl
- link sts3215_03a: geometry collision box size=0.06 0.04 0.07; visual mesh filename=assets/part_4.stl
- link wrist_arm: geometry collision box size=0.07 0.04 0.05; visual mesh filename=assets/sts3215_03a__4.stl
